Commit message: update

File: urdf/cracked_workpiece.urdf (robot description, URDF)
Before this commit: robot crack_block, 2 links, 1 joints
Links:
- link crack_link: geometry collision mesh filename=file:///home/brij/ros2_ws/src/weld_desc/meshes/gazebo_crack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 scale=0.004 0.004 0.004; visual mesh filename=file:///home/brij/ros2_ws/src/weld_desc/meshes/gazebo_crack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 scale=0.004 0.004 0.004
