Commit message: update

File: urdf/weld_robot.xacro (robot description, xacro)
@@ -1,4 +1,4 @@
 <?xml version="1.0"?>
-<robot xmlns:xacro="http://www.ros.org/wiki/xacro" name="weld_robot_ur5e">
+<robot xmlns:xacro="http://www.ros.org/wiki/xacro" name="weld_robot">
   <xacro:arg name="ur_type" default="ur5e" />
   <xacro:include filename="$(find ur_description)/urdf/ur.urdf.xacro" />

File: urdf/weld_torch.xacro (robot description, xacro)
@@ -1,49 +1,54 @@
 <?xml version="1.0"?>
 <robot xmlns:xacro="http://www.ros.org/wiki/xacro">
-    <xacro:macro name="weld_torch" params="prefix parent">
-        <link name="${prefix}torch_base">
-            <visual>
-                <origin xyz="0 0 0.05" rpy="0 0 0"/>
-                <geometry>
-                    <cylinder length="0.1" radius="0.02"/>
-                </geometry>
-                <material name="Grey">
-                    <color rgba="0.5 0.5 0.5 1.0"/>
-                </material>
-            </visual>
-            <collision>
-                <origin xyz="0 0 0.05" rpy="0 0 0"/>
-                <geometry>
-                    <cylinder length="0.1" radius="0.02"/>
-                </geometry>
-            </collision>
-        </link>
-        <link name="${prefix}torch_tip">
-            <visual>
-                <origin xyz="0 0 0.025" rpy="0 0 0"/>
-                <geometry>
-                    <cylinder length="0.05" radius="0.005"/>
-                </geometry>
-                <material name="Copper">
-                    <color rgba="0.8 0.5 0.2 1.0"/>
-                </material>
-            </visual>
-            <collision>
-                <origin xyz="0 0 0.025" rpy="0 0 0"/>
-                <geometry>
-                    <cylinder length="0.05" radius="0.005"/>
-                </geometry>
-            </collision>
-        </link>
-        <joint name="${prefix}base_to_tip_joint" type="fixed">
-            <parent link="${prefix}torch_base"/>
-            <child link="${prefix}torch_tip"/>
-            <origin xyz="0 0 0.1" rpy="0 0 0"/>
-        </joint>
-        <joint name="${prefix}torch_to_robot_joint" type="fixed">
-            <parent link="${parent}"/>
-            <child link="${prefix}torch_base"/>
-            <origin xyz="0 0 0" rpy="0 0 0"/>
-        </joint>
-    </xacro:macro>
+  <xacro:macro name="weld_torch" params="prefix parent">
+    <link name="${prefix}torch_base">
+      <visual>
+        <origin xyz="0 0 0.05" rpy="0 0 0"/>
+        <geometry><cylinder length="0.1" radius="0.02"/></geometry>
+        <material name="Grey"><color rgba="0.5 0.5 0.5 1.0"/></material>
+      </visual>
+      <collision>
+        <origin xyz="0 0 0.05" rpy="0 0 0"/>
+        <geometry><cylinder length="0.1" radius="0.02"/></geometry>
+      </collision>
+    </link>
+    <link name="${prefix}torch_tip">
+      <visual>
+        <origin xyz="0 0 0.025" rpy="0 0 0"/>
+        <geometry><cylinder length="0.05" radius="0.005"/></geometry>
+        <material name="Copper"><color rgba="0.8 0.5 0.2 1.0"/></material>
+      </visual>
+      <collision>
+        <origin xyz="0 0 0.025" rpy="0 0 0"/>
+        <geometry><cylinder length="0.05" radius="0.0015"/></geometry>
+      </collision>
+    </link>
+    <joint name="${prefix}base_to_tip_joint" type="fixed">
+      <parent link="${prefix}torch_base"/>
+      <child link="${prefix}torch_tip"/>
+      <origin xyz="0 0 0.1" rpy="0 0 0"/>
+    </joint>
+    <joint name="${prefix}torch_to_robot_joint" type="fixed">
+      <parent link="${parent}"/>
+      <child link="${prefix}torch_base"/>
+      <origin xyz="0 0 0" rpy="0 0 0"/>
+    </joint>
+    <gazebo reference="${prefix}torch_tip">
+      <visual>
+        <material>
+          <ambient>0.0 0.8 1.0 1.0</ambient>
+          <emissive>0.0 0.8 1.0 1.0</emissive>
+        </material>
+      </visual>
+      <light name="${prefix}arc_light" type="point">
+        <pose>0 0 -0.01 0 0 0</pose> <diffuse>0.1 0.1 1.0 1.0</diffuse>
+        <specular>0.8 0.8 0.8 1.0</specular>
+        <attenuation>
+          <range>0.20</range>      <linear>2.0</linear>    <constant>0.1</constant>
+          <quadratic>2.0</quadratic>
+        </attenuation>
+        <cast_shadows>false</cast_shadows>
+      </light>
+    </gazebo>
+  </xacro:macro>
 </robot>

File: urdf/workpiece.xacro (robot description, xacro)
@@ -1,11 +1,8 @@
 <?xml version="1.0"?>
-<robot xmlns:xacro="http://wiki.ros.org/xacro" name="workpiece">
-  <!-- Properties for each plate -->
-  <xacro:property name="plate_length" value="0.5" /> <!-- 50 cm (X direction) -->
-  <xacro:property name="plate_width" value="0.25" /> <!-- 25 cm (Y direction) -->
-  <xacro:property name="plate_height" value="0.01" /> <!-- 1 cm thick (Z direction) -->
-  <!-- Base link (to fix the plates to the world) -->
+<robot xmlns:xacro="http://www.ros.org/wiki/xacro" name="workpiece">
+  <xacro:property name="plate_length" value="0.5" />
+  <xacro:property name="plate_width" value="0.25" />
+  <xacro:property name="plate_height" value="0.01" />
   <link name="world"/>
-  <!-- ================= PLATE 1 (Left Side) ================= -->
   <link name="plate1_link">
     <visual>
@@ -13,6 +10,6 @@
         <box size="${plate_length} ${plate_width} ${plate_height}"/>
       </geometry>
-      <material name="grey">
-        <color rgba="0.5 0.5 0.5 1.0"/>
+      <material name="DarkGrey">
+        <color rgba="0.2 0.2 0.2 1.0"/>
       </material>
     </visual>
@@ -27,13 +24,12 @@
     </inertial>
   </link>
-  <!-- Joint to fix Plate 1 to the world -->
-  <!-- Position: X=0.7m (in front), Y=0.126m (left), Z=0.5m (up) -->
-  <!-- We leave a 1mm gap from the center, so 0.125 (half_width) + 0.001 (gap) = 0.126 -->
+  <gazebo reference="plate1_link">
+    <material>Gazebo/DarkGrey</material>
+  </gazebo>
   <joint name="plate1_joint" type="fixed">
-    <parent link="world"/>
-    <child link="plate1_link"/>
-    <origin xyz="0.7 0.126 0.5" rpy="0 0 0"/>
+    <parent link="world" />
+    <child link="plate1_link" />
+    <origin xyz="0.35 0.126 0.405" rpy="0 0 0"/>
   </joint>
-  <!-- ================= PLATE 2 (Right Side) ================= -->
   <link name="plate2_link">
     <visual>
@@ -41,5 +37,7 @@
         <box size="${plate_length} ${plate_width} ${plate_height}"/>
       </geometry>
-      <material name="grey"/>
+      <material name="DarkGrey">
+        <color rgba="0.2 0.2 0.2 1.0"/>
+      </material>
     </visual>
     <collision>
@@ -53,10 +51,11 @@
     </inertial>
   </link>
-  <!-- Joint to fix Plate 2 to the world -->
-  <!-- Position: X=0.7m (in front), Y=-0.126m (right), Z=0.5m (up) -->
+  <gazebo reference="plate2_link">
+    <material>Gazebo/DarkGrey</material>
+  </gazebo>
   <joint name="plate2_joint" type="fixed">
-    <parent link="world"/>
+    <parent link="world" />
     <child link="plate2_link"/>
-    <origin xyz="0.7 -0.126 0.5" rpy="0 0 0"/>
+    <origin xyz="0.35 -0.126 0.405" rpy="0 0 0"/>
   </joint>
 </robot>

Commit message: update

File: urdf/weld_robot.xacro (robot description, xacro)
@@ -2,4 +2,5 @@
 <robot xmlns:xacro="http://www.ros.org/wiki/xacro" name="weld_robot">
   <xacro:arg name="ur_type" default="ur5e" />
+  <xacro:arg name="transmission_hw_interface" default="hardware_interface/PositionJointInterface" />
   <xacro:include filename="$(find ur_description)/urdf/ur.urdf.xacro" />
   <xacro:include filename="$(find weld_desc)/urdf/weld_torch.xacro" />

File: urdf/weld_torch.xacro (robot description, xacro)
@@ -8,8 +8,14 @@
         <material name="Grey"><color rgba="0.5 0.5 0.5 1.0"/></material>
       </visual>
+      <!-- Added Collision Geometry -->
       <collision>
         <origin xyz="0 0 0.05" rpy="0 0 0"/>
         <geometry><cylinder length="0.1" radius="0.02"/></geometry>
       </collision>
+      <inertial>
+        <origin xyz="0 0 0.05" rpy="0 0 0"/>
+        <mass value="0.2"/>
+        <inertia ixx="0.0002" ixy="0.0" ixz="0.0" iyy="0.0002" iyz="0.0" izz="0.00005"/>
+      </inertial>
     </link>
     <link name="${prefix}torch_tip">
@@ -19,8 +25,14 @@
         <material name="Copper"><color rgba="0.8 0.5 0.2 1.0"/></material>
       </visual>
+      <!-- Added Collision Geometry -->
       <collision>
         <origin xyz="0 0 0.025" rpy="0 0 0"/>
-        <geometry><cylinder length="0.05" radius="0.0015"/></geometry>
+        <geometry><cylinder length="0.05" radius="0.005"/></geometry>
       </collision>
+      <inertial>
+        <origin xyz="0 0 0.025" rpy="0 0 0"/>
+        <mass value="0.05"/>
+        <inertia ixx="0.00001" ixy="0.0" ixz="0.0" iyy="0.00001" iyz="0.0" izz="0.00001"/>
+      </inertial>
     </link>
     <link name="${prefix}tcp"/>
@@ -31,7 +43,14 @@
         <material name="Black"><color rgba="0.1 0.1 0.1 1.0"/></material>
       </visual>
+      <!-- Added Collision Geometry -->
       <collision>
+        <origin xyz="0 0 0" rpy="0 0 0"/>
         <geometry><box size="0.02 0.04 0.02"/></geometry>
       </collision>
+      <inertial>
+        <origin xyz="0 0 0" rpy="0 0 0"/>
+        <mass value="0.1"/>
+        <inertia ixx="0.00002" ixy="0.0" ixz="0.0" iyy="0.00001" iyz="0.0" izz="0.00002"/>
+      </inertial>
     </link>
     <link name="${prefix}camera_optical_frame"/>
