Commit message: UD

File: config/ur5e/weld.srdf.xacro (robot description, xacro)
@@ -5,11 +5,15 @@
   <xacro:include filename="$(find ur_moveit_config)/srdf/ur_macro.srdf.xacro"/>
   <xacro:ur_srdf name="$(arg name)" prefix="$(arg prefix)"/>
+  <group name="welding_arm">
+    <chain base_link="base_link" tip_link="weld_tcp" />
+  </group>
   <group name="hand">
     <link name="tool0"/>
     <link name="weld_torch_base"/>
     <link name="weld_torch_tip"/>
+    <link name="weld_tcp"/>
   </group>
   <group name="end_effector">
-    <link name="weld_torch_tip"/>
+    <link name="weld_tcp"/>
   </group>
   <disable_collisions link1="tool0" link2="weld_torch_base" reason="Adjacent"/>
